File: hardware/kicad/circuitBuilderAi-Astra.kicad_sch (KiCad schematic)
At the start: 0 parts

Commit message: phase4
Connections:
- no-connect marks 5 -> 11
Other:
- sheet 2 - Power Regulation / Sequencing ports: added 12V_PROTECTED, 1V0_DSP_CORE, 1V35_DSP_DMC, 1V8_DSP_REF_ANA, 2V8_MIC, 3V3_ADC_A, 3V3_SYS, 3V8_PRE, 5V_AFE, AFE_EN_CMD, DSP_WDI, EFUSE_FLT_N, PGOOD_12V, POWER_GND, RAILS_OK, SYS_HWRST; removed none
- note added: "4B BLOCKED - rails entered; safe-state / shutdown incomplete"
- note added: "Sheet 1 / Sheet 2 power interfaces connected. Future consumer interfaces terminate here. No PCB."
- note added: "Sheet 1: Phase 4A PASS. Sheet 2: Phase 4B BLOCKED, partial entry. Sheets 3-7: placeholders."
- note removed: "PHASE 4A - Sheet 1 implemented to Phase 3A; Sheets 2-7 remain placeholders."
- note removed: "Sheet 1 interfaces terminate here until later-phase authorization. No PCB created."
Changed lines of the file:
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@@
 		(title "circuitBuilderAi-Astra - Schematic Hierarchy")
 		(date "2026-09-09")
-		(rev "4A")
+		(rev "4B-BLOCKED")
 		(company "circuitBuilderAi-Astra")
-		(comment 1 "Sheet 1 only. Later circuitry and PCB implementation are not authorized.")
+		(comment 1 "Sheet 2 partially entered; Phase 4B BLOCKED. Later circuitry remains unimplemented.")
 	)
 	(text "PLACEHOLDER - not implemented in Phase 4A"
@@
 		)
 	)
+	(text "4B BLOCKED - rails entered; safe-state / shutdown incomplete"
+		(exclude_from_sim no)
+		(at 225 56 0)
+		(effects
+			(font
+				(size 1.5 1.5)
+			)
+			(justify left bottom)
+		)
+	)
+	(text "Phase 3 section 14: seven logical sheets. Root is KiCad page 1; logical sheets 1-7 are pages 2-8."
+		(exclude_from_sim no)
+		(at 25 35 0)
+		(effects
+			(font
+				(size 1.5 1.5)
+			)
+			(justify left bottom)
+		)
+	)
+	(text "Sheet 1 / Sheet 2 power interfaces connected. Future consumer interfaces terminate here. No PCB."
+		(exclude_from_sim no)
+		(at 25 43 0)
+		(effects
+			(font
+				(size 1.5 1.5)
+			)
+			(justify left bottom)
+		)
+	)
+	(text "Sheet 1: Phase 4A PASS. Sheet 2: Phase 4B BLOCKED, partial entry. Sheets 3-7: placeholders."
+		(exclude_from_sim no)
+		(at 25 25 0)
+		(effects
+			(font
+				(size 2 2)
+			)
+			(justify left bottom)
+		)
+	)
 	(text "PLACEHOLDER - not implemented in Phase 4A"
 		(exclude_from_sim no)
-		(at 230 80 0)
-		(effects
-			(font
-				(size 1.5 1.5)
-			)
-			(justify left bottom)
-		)
-	)
-	(text "Phase 3 section 14: seven logical sheets. Root is KiCad page 1; logical sheets 1-7 are pages 2-8."
-		(exclude_from_sim no)
-		(at 25 35 0)
-		(effects
-			(font
-				(size 1.5 1.5)
-			)
-			(justify left bottom)
-		)
-	)
-	(text "Sheet 1 interfaces terminate here until later-phase authorization. No PCB created."
-		(exclude_from_sim no)
-		(at 25 43 0)
-		(effects
-			(font
-				(size 1.5 1.5)
-			)
-			(justify left bottom)
-		)
-	)
-	(text "PHASE 4A - Sheet 1 implemented to Phase 3A; Sheets 2-7 remain placeholders."
-		(exclude_from_sim no)
-		(at 25 25 0)
-		(effects
-			(font
-				(size 2 2)
-			)
-			(justify left bottom)
-		)
-	)
-	(text "PLACEHOLDER - not implemented in Phase 4A"
-		(exclude_from_sim no)
 		(at 30 221 0)
 		(effects
@@
 	)
 	(no_connect
-		(at 195 77.7)
-	)
-	(no_connect
-		(at 195 85.32)
-	)
-	(no_connect
-		(at 195 81.51)
-	)
-	(no_connect
-		(at 195 73.89)
-	)
-	(no_connect
-		(at 195 70.08)
+		(at 395 73.89)
+	)
+	(no_connect
+		(at 225 92.94)
+	)
+	(no_connect
+		(at 395 70.08)
+	)
+	(no_connect
+		(at 395 100.56)
+	)
+	(no_connect
+		(at 395 77.7)
+	)
+	(no_connect
+		(at 395 89.13)
+	)
+	(no_connect
+		(at 395 96.75)
+	)
+	(no_connect
+		(at 395 85.32)
+	)
+	(no_connect
+		(at 395 81.51)
+	)
+	(no_connect
+		(at 395 92.94)
+	)
+	(no_connect
+		(at 225 89.13)
+	)
+	(wire
+		(pts
+			(xy 195 85.32) (xy 225 85.32)
+		)
+		(stroke
+			(width 0)
+			(type default)
+		)
+	)
+	(wire
+		(pts
+			(xy 195 73.89) (xy 225 73.89)
+		)
+		(stroke
+			(width 0)
+			(type default)
+		)
+	)
+	(wire
+		(pts
+			(xy 195 81.51) (xy 225 81.51)
+		)
+		(stroke
+			(width 0)
+			(type default)
+		)
+	)
+	(wire
+		(pts
+			(xy 195 77.7) (xy 225 77.7)
+		)
+		(stroke
+			(width 0)
+			(type default)
+		)
+	)
+	(wire
+		(pts
+			(xy 195 70.08) (xy 225 70.08)
+		)
+		(stroke
+			(width 0)
+			(type default)
+		)
 	)
 	(sheet
@@
 	(sheet
 		(at 225 65)
-		(size 170 27)
+		(size 170 38.1)
 		(exclude_from_sim no)
 		(in_bom yes)
@@
 		)
 		(property "Sheetfile" "power_regulation.kicad_sch"
-			(at 225 93.5 0)
+			(at 225 104.6 0)
 			(show_name no)
 			(do_not_autoplace no)
@@
 			)
 		)
+		(pin "12V_PROTECTED" input
+			(at 225 70.08 180)
+			(effects
+				(font
+					(size 1.016 1.016)
+				)
+			)
+		)
+		(pin "POWER_GND" passive
+			(at 225 73.89 180)
+			(effects
+				(font
+					(size 1.016 1.016)
+				)
+			)
+		)
+		(pin "3V8_PRE" output
+			(at 225 77.7 180)
+			(effects
+				(font
+					(size 1.016 1.016)
+				)
+			)
+		)
+		(pin "PGOOD_12V" input
+			(at 225 81.51 180)
+			(effects
+				(font
+					(size 1.016 1.016)
+				)
+			)
+		)
+		(pin "EFUSE_FLT_N" input
+			(at 225 85.32 180)
+			(effects
+				(font
+					(size 1.016 1.016)
+				)
+			)
+		)
+		(pin "DSP_WDI" input
+			(at 225 89.13 180)
+			(effects
+				(font
+					(size 1.016 1.016)
+				)
+			)
+		)
+		(pin "AFE_EN_CMD" input
+			(at 225 92.94 180)
+			(effects
+				(font
+					(size 1.016 1.016)
+				)
+			)
+		)
+		(pin "1V8_DSP_REF_ANA" output
+			(at 395 70.08 0)
+			(effects
+				(font
+					(size 1.016 1.016)
+				)
+			)
+		)
+		(pin "1V0_DSP_CORE" output
+			(at 395 73.89 0)
+			(effects
+				(font
+					(size 1.016 1.016)
+				)
+			)
+		)
+		(pin "1V35_DSP_DMC" output
+			(at 395 77.7 0)
+			(effects
+				(font
+					(size 1.016 1.016)
+				)
+			)
+		)
+		(pin "3V3_SYS" output
+			(at 395 81.51 0)
+			(effects
+				(font
+					(size 1.016 1.016)
+				)
+			)
+		)
+		(pin "3V3_ADC_A" output
+			(at 395 85.32 0)
+			(effects
+				(font
+					(size 1.016 1.016)
+				)
+			)
+		)
+		(pin "2V8_MIC" output
+			(at 395 89.13 0)
+			(effects
+				(font
+					(size 1.016 1.016)
+				)
+			)
+		)
+		(pin "5V_AFE" output
+			(at 395 92.94 0)
+			(effects
+				(font
+					(size 1.016 1.016)
+				)
+			)
+		)
+		(pin "RAILS_OK" output
+			(at 395 96.75 0)
+			(effects
+				(font
+					(size 1.016 1.016)
+				)
+			)
+		)
+		(pin "SYS_HWRST" bidirectional
+			(at 395 100.56 0)
+			(effects
+				(font
+					(size 1.016 1.016)
+				)
+			)
+		)

Commit message: phase 4c
Connections:
- no-connect marks 11 -> 57
Other:
- sheet 2 - Power Regulation / Sequencing ports: added ADC_AIN1N, ADC_AIN1P, ADC_AIN2N, ADC_AIN2P, ADC_AIN3N, ADC_AIN3P, ADC_AIN4N, ADC_AIN4P, ADC_PD_RST_N, ADC_RST_RELEASE_CMD, ADC_VREF, AFE1N_AFTER_47R, AFE1P_AFTER_47R, AFE1_BEFORE_4u7, AFE2N_AFTER_47R, AFE2P_AFTER_47R, AFE2_BEFORE_4u7, AFE3N_AFTER_47R, AFE3P_AFTER_47R, AFE3_BEFORE_4u7, AFE4N_AFTER_47R, AFE4P_AFTER_47R, AFE4_BEFORE_4u7, AFE_VCM_INPUT, AMP_FAULT_N, AMP_MUTE_CMD, AMP_MUTE_RELEASE, AMP_STBY_CMD, AMP_STBY_RELEASE, ANALOG_PWR_CMD, ANALOG_PWR_EN, AUDIO_CLOCK_OE_N, AUDIO_DATA_OE_CMD, AUDIO_DATA_OE_N, CLOCK_STARTUP_CMD, CLOCK_STARTUP_EN, HW_RUN_LATCHED, MCLK_OE_N, MIC1_AFTER_100R, MIC2_AFTER_100R, MIC3_AFTER_100R, MIC4_AFTER_100R, RUN_HEALTH_OK_3V8, RUN_HEALTH_OK_CMD, SAFE_ARM_CMD, SAFE_CLEAR_N, SHUTDOWN_REQ; removed AFE_EN_CMD
- note added: "Sheet 1: Phase 4A. Sheet 2: regulation / retained sequencing / bootstrap controls. Sheets 3-7: future endpoints."
- note added: "Sheet 2: Phase 3D/3E/3F implementation; validation record controls gate"
- note removed: "4B BLOCKED - rails entered; safe-state / shutdown incomplete"
- note removed: "Sheet 1: Phase 4A PASS. Sheet 2: Phase 4B BLOCKED, partial entry. Sheets 3-7: placeholders."

Commit message: before-rebuilding
Last changes before rebuilding PCB design
Connections:
- no-connect marks 57 -> 65
Other:
- sheet 2 - Power Regulation / Sequencing ports: added ADC1_N_ISO, ADC1_P_ISO, ADC2_N_ISO, ADC2_P_ISO, ADC3_N_ISO, ADC3_P_ISO, ADC4_N_ISO, ADC4_P_ISO, ADC_VREF_RAW, AFE1_N_RAW, AFE1_P_RAW, AFE2_N_RAW, AFE2_P_RAW, AFE3_N_RAW, AFE3_P_RAW, AFE4_N_RAW, AFE4_P_RAW, AFE_VCM_ISO, MIC1_N_ISO, MIC1_N_RAW, MIC1_P_ISO, MIC1_P_RAW, MIC2_N_ISO, MIC2_N_RAW, MIC2_P_ISO, MIC2_P_RAW, MIC3_N_ISO, MIC3_N_RAW, MIC3_P_ISO, MIC3_P_RAW, MIC4_N_ISO, MIC4_N_RAW, MIC4_P_ISO, MIC4_P_RAW; removed ADC_AIN1N, ADC_AIN1P, ADC_AIN2N, ADC_AIN2P, ADC_AIN3N, ADC_AIN3P, ADC_AIN4N, ADC_AIN4P, ADC_VREF, AFE1N_AFTER_47R, AFE1P_AFTER_47R, AFE1_BEFORE_4u7, AFE2N_AFTER_47R, AFE2P_AFTER_47R, AFE2_BEFORE_4u7, AFE3N_AFTER_47R, AFE3P_AFTER_47R, AFE3_BEFORE_4u7, AFE4N_AFTER_47R, AFE4P_AFTER_47R, AFE4_BEFORE_4u7, AFE_VCM_INPUT, MIC1_AFTER_100R, MIC2_AFTER_100R, MIC3_AFTER_100R, MIC4_AFTER_100R
Changed lines of the file:
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@@
+	)
+	(no_connect
+		(at 800 314.96)
 	)
 	(no_connect
@@
 	)
 	(no_connect
+		(at 800 309.88)
+	)
+	(no_connect
 		(at 800 284.48)
 	)
@@
 	)
 	(no_connect
+		(at 800 320.04)
+	)
+	(no_connect
 		(at 800 299.72)
 	)
@@
 	)
 	(no_connect
+		(at 800 304.8)
+	)
+	(no_connect
 		(at 800 254)
 	)
@@
 	)
 	(no_connect
+		(at 800 330.2)
+	)
+	(no_connect
 		(at 800 101.6)
 	)
@@
 	)
 	(no_connect
+		(at 800 335.28)
+	)
+	(no_connect
 		(at 800 259.08)
 	)
@@
 	)
 	(no_connect
+		(at 800 340.36)
+	)
+	(no_connect
 		(at 800 81.28)
+	)
+	(no_connect
+		(at 800 325.12)
 	)
 	(wire
@@
 			)
 		)
-		(pin "AFE1P_AFTER_47R" passive
+		(pin "AFE1_P_RAW" passive
 			(at 800 172.72 0)
 			(effects
@@
 			)
 		)
-		(pin "ADC_AIN1P" passive
+		(pin "ADC1_P_ISO" passive
 			(at 800 177.8 0)
 			(effects
@@
 			)
 		)
-		(pin "AFE1N_AFTER_47R" passive
+		(pin "AFE1_N_RAW" passive
 			(at 800 182.88 0)
 			(effects
@@
 			)
 		)
-		(pin "ADC_AIN1N" passive
+		(pin "ADC1_N_ISO" passive
 			(at 800 187.96 0)
 			(effects
@@
 			)
 		)
-		(pin "AFE2P_AFTER_47R" passive
+		(pin "AFE2_P_RAW" passive
 			(at 800 193.04 0)
 			(effects
@@
 			)
 		)
-		(pin "ADC_AIN2P" passive
+		(pin "ADC2_P_ISO" passive
 			(at 800 198.12 0)
 			(effects
@@
 			)
 		)
-		(pin "AFE2N_AFTER_47R" passive
+		(pin "AFE2_N_RAW" passive
 			(at 800 203.2 0)
 			(effects
@@
 			)
 		)
-		(pin "ADC_AIN2N" passive
+		(pin "ADC2_N_ISO" passive
 			(at 800 208.28 0)
 			(effects
@@
 			)
 		)
-		(pin "AFE3P_AFTER_47R" passive
+		(pin "AFE3_P_RAW" passive
 			(at 800 213.36 0)
 			(effects
@@
 			)
 		)
-		(pin "ADC_AIN3P" passive
+		(pin "ADC3_P_ISO" passive
 			(at 800 218.44 0)
 			(effects
@@
 			)
 		)
-		(pin "AFE3N_AFTER_47R" passive
+		(pin "AFE3_N_RAW" passive
 			(at 800 223.52 0)
 			(effects
@@
 			)
 		)
-		(pin "ADC_AIN3N" passive
+		(pin "ADC3_N_ISO" passive
 			(at 800 228.6 0)
 			(effects
@@
 			)
 		)
-		(pin "AFE4P_AFTER_47R" passive
+		(pin "AFE4_P_RAW" passive
 			(at 800 233.68 0)
 			(effects
@@
 			)
 		)
-		(pin "ADC_AIN4P" passive
+		(pin "ADC4_P_ISO" passive
 			(at 800 238.76 0)
 			(effects
@@
 			)
 		)
-		(pin "AFE4N_AFTER_47R" passive
+		(pin "AFE4_N_RAW" passive
 			(at 800 243.84 0)
 			(effects
@@
 			)
 		)
-		(pin "ADC_AIN4N" passive
+		(pin "ADC4_N_ISO" passive
 			(at 800 248.92 0)
 			(effects
@@
 			)
 		)
-		(pin "ADC_VREF" passive
+		(pin "ADC_VREF_RAW" passive
 			(at 800 254 0)
 			(effects
@@
 			)
 		)
-		(pin "AFE_VCM_INPUT" passive
+		(pin "AFE_VCM_ISO" passive
 			(at 800 259.08 0)
 			(effects
@@
 			)
 		)
-		(pin "MIC1_AFTER_100R" passive
+		(pin "MIC1_P_RAW" passive
 			(at 800 264.16 0)
 			(effects
@@
 			)
 		)
-		(pin "AFE1_BEFORE_4u7" passive
+		(pin "MIC1_P_ISO" passive
 			(at 800 269.24 0)
 			(effects
@@
 			)
 		)
-		(pin "MIC2_AFTER_100R" passive
+		(pin "MIC2_P_RAW" passive
 			(at 800 274.32 0)
 			(effects
@@
 			)
 		)
-		(pin "AFE2_BEFORE_4u7" passive
+		(pin "MIC2_P_ISO" passive
 			(at 800 279.4 0)
 			(effects
@@
 			)
 		)
-		(pin "MIC3_AFTER_100R" passive
+		(pin "MIC3_P_RAW" passive
 			(at 800 284.48 0)
 			(effects
@@
 			)
 		)
-		(pin "AFE3_BEFORE_4u7" passive
+		(pin "MIC3_P_ISO" passive
 			(at 800 289.56 0)
 			(effects
@@
 			)
 		)
-		(pin "MIC4_AFTER_100R" passive
+		(pin "MIC4_P_RAW" passive
 			(at 800 294.64 0)
 			(effects
@@
 			)
 		)
-		(pin "AFE4_BEFORE_4u7" passive
+		(pin "MIC4_P_ISO" passive
 			(at 800 299.72 0)
 			(effects
 				(font
+					(size 1.016 1.016)
+				)
+			)
+		)
+		(pin "MIC1_N_RAW" passive
+			(at 800 304.8 0)
+			(effects
+				(font
+					(size 1.016 1.016)
+				)
+			)
+		)
+		(pin "MIC2_N_RAW" passive
+			(at 800 309.88 0)
+			(effects
+				(font
+					(size 1.016 1.016)
+				)
+			)
+		)
+		(pin "MIC3_N_RAW" passive
+			(at 800 314.96 0)
+			(effects
+				(font
+					(size 1.016 1.016)
+				)
+			)
+		)
+		(pin "MIC4_N_RAW" passive
+			(at 800 320.04 0)
+			(effects
+				(font
+					(size 1.016 1.016)
+				)
+			)
+		)
+		(pin "MIC1_N_ISO" passive
+			(at 800 325.12 0)
+			(effects
+				(font
+					(size 1.016 1.016)
+				)
+			)
+		)
+		(pin "MIC2_N_ISO" passive
+			(at 800 330.2 0)
+			(effects
+				(font
+					(size 1.016 1.016)
+				)
+			)
+		)
+		(pin "MIC3_N_ISO" passive
+			(at 800 335.28 0)
+			(effects
+				(font
+					(size 1.016 1.016)
+				)
+			)
+		)
+		(pin "MIC4_N_ISO" passive
+			(at 800 340.36 0)
+			(effects
+				(font
