File: hardware/kicad/power_regulation.kicad_sch (KiCad schematic)
At the start: 0 parts

Commit message: phase4
Parts:
- added C201, C211, C221, C231, C232, C236, C241, C242, C246, C251, C252, C256, C261, C262, C271, C272: 10u, Capacitor_SMD:C_1206_3216Metric, symbol Astra_Sequencing:C
- added C202, C212, C222, C234, C244, C253, C254: 10n, Capacitor_SMD:C_0603_1608Metric, symbol Astra_Sequencing:C
- added C203, C204, C206, C216, C223, C224, C226: 22u, Capacitor_SMD:C_1206_3216Metric, symbol Astra_Sequencing:C
- added C213, C214, C215, C245: 47u, Capacitor_SMD:C_1206_3216Metric, symbol Astra_Sequencing:C
- added C233, C243: 47n, Capacitor_SMD:C_0603_1608Metric, symbol Astra_Sequencing:C
- added C263, C273, C281, C282, C283: 100n, Capacitor_SMD:C_0603_1608Metric, symbol Astra_Sequencing:C
- added L201, L202, L203: 1u, Inductor_SMD:L_Coilcraft_XAL4020-XXX, symbol Astra_Sequencing:L
- added R201: 44.2k, Resistor_SMD:R_0603_1608Metric, symbol Astra_Sequencing:R
- added R202, R212, R222, R281, R282, R283, R284, R292, R295, R298, R301: 10.0k, Resistor_SMD:R_0603_1608Metric, symbol Astra_Sequencing:R
- added R211: 4.32k, Resistor_SMD:R_0603_1608Metric, symbol Astra_Sequencing:R
- added R221: 37.1k, Resistor_SMD:R_0603_1608Metric, symbol Astra_Sequencing:R
- added R231: 54.2k, Resistor_SMD:R_0603_1608Metric, symbol Astra_Sequencing:R
- added R232: 100, Resistor_SMD:R_0603_1608Metric, symbol Astra_Sequencing:R
- added R233, R243, R253, R310: 100k, Resistor_SMD:R_0603_1608Metric, symbol Astra_Sequencing:R
- added R234: 1.69k, Resistor_SMD:R_0603_1608Metric, symbol Astra_Sequencing:R
- added R241: 14.9k, Resistor_SMD:R_0603_1608Metric, symbol Astra_Sequencing:R
- added R244: 1.24k, Resistor_SMD:R_0603_1608Metric, symbol Astra_Sequencing:R
- added R251: 324k, Resistor_SMD:R_0603_1608Metric, symbol Astra_Sequencing:R
- added R254: 4.70k, Resistor_SMD:R_0603_1608Metric, symbol Astra_Sequencing:R
- added R261: 3.01k, Resistor_SMD:R_0603_1608Metric, symbol Astra_Sequencing:R
- added R271: 2.55k, Resistor_SMD:R_0603_1608Metric, symbol Astra_Sequencing:R
- added R285: 1.0M, Resistor_SMD:R_0603_1608Metric, symbol Astra_Sequencing:R
- added R291: 24.9k, Resistor_SMD:R_0603_1608Metric, symbol Astra_Sequencing:R
- added R294: 9.31k, Resistor_SMD:R_0603_1608Metric, symbol Astra_Sequencing:R
- added R297: 15.8k, Resistor_SMD:R_0603_1608Metric, symbol Astra_Sequencing:R
- added R300: 53.6k, Resistor_SMD:R_0603_1608Metric, symbol Astra_Sequencing:R
- added R303: 280, Resistor_SMD:R_0603_1608Metric, symbol Astra_Sequencing:R
- added TP201: 3V8_PRE, symbol Astra_Sequencing:TestPoint
- added TP202: 3V8_PRE_FB, symbol Astra_Sequencing:TestPoint
- added TP203: 3V8_PRE_SS, symbol Astra_Sequencing:TestPoint
- added TP204: 1V0_DSP_CORE, symbol Astra_Sequencing:TestPoint
- added TP205: 1V0_DSP_CORE_FB, symbol Astra_Sequencing:TestPoint
- added TP206: 1V0_DSP_CORE_SS, symbol Astra_Sequencing:TestPoint
- added TP207: 3V3_SYS, symbol Astra_Sequencing:TestPoint
- added TP208: 3V3_SYS_FB, symbol Astra_Sequencing:TestPoint
- added TP209: 3V3_SYS_SS, symbol Astra_Sequencing:TestPoint
- added TP210: 1V8_DSP_REF_ANA, symbol Astra_Sequencing:TestPoint
- added TP211: 1V8_DSP_REF_ANA_FB, symbol Astra_Sequencing:TestPoint
- added TP212: 1V8_DSP_REF_ANA_NR, symbol Astra_Sequencing:TestPoint
- added TP213: 1V35_DSP_DMC, symbol Astra_Sequencing:TestPoint
- added TP214: 1V35_DSP_DMC_FB, symbol Astra_Sequencing:TestPoint
- added TP215: 1V35_DSP_DMC_NR, symbol Astra_Sequencing:TestPoint
- added TP216: 5V_AFE, symbol Astra_Sequencing:TestPoint
- added TP217: 5V_AFE_FB, symbol Astra_Sequencing:TestPoint
- added TP218: 5V_AFE_NR, symbol Astra_Sequencing:TestPoint
- added TP219: 3V3_ADC_A, symbol Astra_Sequencing:TestPoint
- added TP220: 2V8_MIC, symbol Astra_Sequencing:TestPoint
- added TP221: SENSE_1V8, symbol Astra_Sequencing:TestPoint
- added TP222: SENSE_CORE, symbol Astra_Sequencing:TestPoint
- added TP223: SENSE_DMC, symbol Astra_Sequencing:TestPoint
- added TP224: SENSE_3V3, symbol Astra_Sequencing:TestPoint
- added TP225: RAILS_OK, symbol Astra_Sequencing:TestPoint
- added TP226: SYS_HWRST, symbol Astra_Sequencing:TestPoint
- added TP227: OUT1, symbol Astra_Sequencing:TestPoint
- added TP228: DSP_WDI, symbol Astra_Sequencing:TestPoint
- added TP229: EN_3V3_SYS, symbol Astra_Sequencing:TestPoint
- added TP230: AFE_EN, symbol Astra_Sequencing:TestPoint
- added TP231: PGOOD_12V, symbol Astra_Sequencing:TestPoint
- added TP232: EFUSE_FLT_N, symbol Astra_Sequencing:TestPoint
- added TP233: 12V_PROTECTED, symbol Astra_Sequencing:TestPoint
- added TP234: POWER_GND, symbol Astra_Sequencing:TestPoint
- added TP235: SUP_REF, symbol Astra_Sequencing:TestPoint
- added TP236: AFE_EN_CMD, symbol Astra_Sequencing:TestPoint
- added U201, U202, U203: TPS62135RGXR, Astra_Sequencing:Texas_RGX0011A, symbol Astra_Sequencing:TPS62135RGXR
- added U204, U205, U206: TPS7A4901DGNR, Package_SO:Texas_DGN0008D_VSSOP-8-1EP_3x3mm_P0.65mm_EP2x2.94mm_Mask1.57x1.89mm, symbol Astra_Sequencing:TPS7A4901DGNR
- added U207: TPS7A2033PDBVR, Package_TO_SOT_SMD:SOT-23-5, symbol Astra_Sequencing:TPS7A2033PDBVR
- added U208: TPS7A2028PDBVR, Package_TO_SOT_SMD:SOT-23-5, symbol Astra_Sequencing:TPS7A2028PDBVR
- added U209: LTC2964HUDC#PBF, Package_DFN_QFN:QFN-20-1EP_3x4mm_P0.5mm_EP1.65x2.65mm, symbol Astra_Sequencing:LTC2964HUDC_PBF
- added U210: TPS3431SDRBR, Package_DFN_QFN:Texas_DRB0008A, symbol Astra_Sequencing:TPS3431SDRBR
- added U211: SN74LV1T08DBVR, Package_TO_SOT_SMD:SOT-23-5, symbol Astra_Sequencing:SN74LV1T08DBVR
Connections:
- new net 12V_PROTECTED: C201.1, C221.1, C251.1, TP233.1, U201.1 (VIN), U201.10 (MODE), U201.8 (EN), U203.1 (VIN), U203.10 (MODE), U206.8 (IN)
- new net 1V0_DSP_CORE: C213.1, C214.1, C215.1, C216.1, L202.2, R211.1, R294.1, TP204.1, U202.6 (VOS)
- new net 1V0_DSP_CORE_FB: R211.2, R212.1, TP205.1, U202.5 (FB)
- new net 1V0_DSP_CORE_SS: C212.1, TP206.1, U202.9 (SS/TR)
- new net 1V0_DSP_CORE_SW: L202.1, U202.2 (SW)
- new net 1V35_DSP_DMC: C242.1, C244.1, C245.1, C246.1, R241.1, R244.1, R297.1, TP213.1, U205.1 (OUT)
- new net 1V35_DSP_DMC_FB: C244.2, R241.2, R243.1, TP214.1, U205.2 (FB)
- new net 1V35_DSP_DMC_NR: C243.1, TP215.1, U205.6 (NR/SS)
- new net 1V8_DSP_REF_ANA: C232.1, C234.1, C236.1, R231.1, R234.1, R291.1, TP210.1, U204.1 (OUT)
- new net 1V8_DSP_REF_ANA_FB: C234.2, R232.2, R233.1, TP211.1, U204.2 (FB)
- new net 1V8_DSP_REF_ANA_FB_TOP_MID: R231.2, R232.1
- new net 1V8_DSP_REF_ANA_NR: C233.1, TP212.1, U204.6 (NR/SS)
- new net 2V8_MIC: C272.1, C273.1, R271.1, TP220.1, U208.5 (OUT)
- new net 3V3_ADC_A: C262.1, C263.1, R261.1, TP219.1, U207.5 (OUT)
- new net 3V3_SYS: C223.1, C224.1, C226.1, C282.1, L203.2, R221.1, R282.1, R283.1, R300.1, TP207.1, U203.6 (VOS), U210.1 (VDD), U210.5 (SET1)
- new net 3V3_SYS_FB: R221.2, R222.1, TP208.1, U203.5 (FB)
- new net 3V3_SYS_SS: C222.1, TP209.1, U203.9 (SS/TR)
- new net 3V3_SYS_SW: L203.1, U203.2 (SW)
- new net 3V8_PRE: C203.1, C204.1, C206.1, C211.1, C231.1, C241.1, C261.1, C271.1, C281.1, C283.1, L201.2, R201.1, R281.1, TP201.1, U201.6 (VOS), U202.1 (VIN), U202.10 (MODE), U204.8 (IN), U205.8 (IN), U207.1 (IN), U208.1 (IN), U209.1 (RDIS), U209.11 (RT), U209.2 (MR), U209.4 (VCC), U211.5 (VCC)
- new net 3V8_PRE_FB: R201.2, R202.1, TP202.1, U201.5 (FB)
- new net 3V8_PRE_SS: C202.1, TP203.1, U201.9 (SS/TR)
- new net 3V8_PRE_SW: L201.1, U201.2 (SW)
- new net 5V_AFE: C252.1, C254.1, C256.1, R251.1, R254.1, TP216.1, U206.1 (OUT)
- new net 5V_AFE_FB: C254.2, R251.2, R253.1, TP217.1, U206.2 (FB)
- new net 5V_AFE_NR: C253.1, TP218.1, U206.6 (NR/SS)
- new net AFE_EN: R310.1, TP230.1, U206.5 (EN)
- new net AFE_EN_CMD: TP236.1
- new net DSP_WDI: R284.1, TP228.1, U210.6 (WDI)
- new net EFUSE_FLT_N: TP232.1
- new net EN_3V3_SYS: R285.1, TP229.1, U203.8 (EN), U211.4 (Y)
- new net OUT1: R281.2, TP227.1, U202.8 (EN), U205.5 (EN), U207.3 (EN), U208.3 (EN), U209.7 (OUT1), U211.1 (A)
- new net PGOOD_12V: TP231.1, U204.5 (EN), U211.2 (B)
- new net POWER_GND: C201.2, C202.2, C203.2, C204.2, C206.2, C211.2, C212.2, C213.2, C214.2, C215.2, C216.2, C221.2, C222.2, C223.2, C224.2, C226.2, C231.2, C232.2, C233.2, C236.2, C241.2, C242.2, C243.2, C245.2, C246.2, C251.2, C252.2, C253.2, C256.2, C261.2, C262.2, C263.2, C271.2, C272.2, C273.2, C281.2, C282.2, C283.2, R202.2, R212.2, R222.2, R233.2, R234.2, R243.2, R244.2, R253.2, R254.2, R261.2, R271.2, R284.2, R285.2, R292.2, R295.2, R298.2, R301.2, R310.2, TP234.1, U201.11 (VSEL), U201.3 (GND), U201.4 (FB2), U202.11 (VSEL), U202.3 (GND), U202.4 (FB2), U203.11 (VSEL), U203.3 (GND), U203.4 (FB2), U204.4 (GND), U204.9 (EP), U205.4 (GND), U205.9 (EP), U206.4 (GND), U206.9 (EP), U207.2 (GND), U208.2 (GND), U209.21 (EP), U209.3 (DVCC), U209.6 (GND), U210.4 (GND), U210.9 (EP), U211.3 (GND)
- new net RAILS_OK: R282.2, TP225.1, U209.5 (RST), U210.3 (EN)
- new net SENSE_1V8: R291.2, R292.1, TP221.1, U209.20 (V1)
- new net SENSE_3V3: R300.2, R301.1, TP224.1, U209.17 (V4)
- new net SENSE_CORE: R294.2, R295.1, TP222.1, U209.19 (V2)
- new net SENSE_DMC: R298.1, R303.2, TP223.1, U209.18 (V3)
- new net SENSE_DMC_MID: R297.2, R303.1
- new net SUP_REF: TP235.1, U209.12 (PG4), U209.13 (PG3), U209.14 (PG2), U209.15 (PG1), U209.16 (REF)
- new net SYS_HWRST: R283.2, TP226.1, U210.7 (WDO), U210.8 (ENOUT)
- no-connect marks 0 -> 15
Other:
- note added: "1V0_DSP_CORE | TPS62135 forced PWM"
- note added: "1V35_DSP_DMC | TPS7A4901DGNR"
- note added: "1V8_DSP_REF_ANA | TPS7A4901DGNR"
- note added: "2V8_MIC | TPS7A2028PDBVR"
- note added: "3V3_ADC_A | TPS7A2033PDBVR"
- note added: "3V3_SYS EN = OUT1 AND PGOOD_12V 1.0M EN pulldown; inputs remain separate status nets."
- note added: "3V3_SYS | TPS62135 forced PWM"
- note added: "3V8_PRE | TPS62135 forced PWM"
- note added: "5V_AFE | TPS7A4901DGNR"
- note added: "AFE EN held off by R310. Command and fault override NOT connected. No power-up / reset / safe-state implementation approval is implied. Hardware-safe latch, dominance, commanded shutdown, and AFE override are incomplete."
- note added: "CWD NC; SET1=VDD; WDO and ENOUT wired open drain. 330..470ms total rail-valid to reset release; WDT 1.36..1.84s. First DSP falling WDI edge <=1.13s after reset release. DSP WDI default low; firmware services during boot."
- note added: "DNC pin 7 and NC pin 3 open; EP pin 9 grounded. Preload is permanent, included in total rail allocation. CFF spans OUT to FB (including series top-arm resistors)."
- note added: "Four DSP rail comparators / first-rail qualification"
- note added: "MODE=VIN; VSEL=0; FB2=0; native PG intentionally NC. Kelvin FB bottom to GND; VOS to local COUT positive. L/C qualification and distributed capacitance remain board validation."
- note added: "P variant: active output discharge. EN=OUT1. No startup-time guarantee extrapolated to this capacitor bank. Consumer-side filtering/decoupling belongs to the later load sheets."
- note added: "PG1..PG4 = REF (+ADJ); no PG capacitors. RT=VCC: 160..240ms. RST=RAILS_OK, isolated from SYS_HWRST. Do not substitute regulator PG; sense returns Kelvin to supervisor GND."
- note added: "PHASE 4B BLOCKED: common OUT1 cannot turn microphones off while retaining core/DMC power. Phase 3D section 9.1(5), 11(6) versus section 9.2 commanded-shutdown order. No enable relation changed."
- note added: "TPS3431: independent watchdog / delayed reset"
- note removed: "2 - Power Regulation / Sequencing"
- note removed: "INTENTIONALLY UNIMPLEMENTED - hierarchy placeholder only."
- note removed: "No components, nets, or speculative hierarchical signals. Implementation requires later phase authorization."

Commit message: phase 4c
Parts:
- removed C283: 100n, Capacitor_SMD:C_0603_1608Metric, symbol Astra_Sequencing:C
- removed R285: 1.0M, Resistor_SMD:R_0603_1608Metric, symbol Astra_Sequencing:R
- added C300, C301, C302, C303, C304, C305, C306, C307, C308, C309, C310, C311, C312, C313, C314, C315, C316, C317, C318, C341, C350, C351, C352, C353, C354, C355, C356, C357, C358, C359, C360, C361, C362, C363: 100n, Capacitor_SMD:C_0603_1608Metric, symbol Astra_Sequencing:C
- added C340: 220n, Capacitor_SMD:C_1210_3225Metric, symbol Astra_Sequencing:C
- added Q201, Q202, Q203: BSS138LT1G, Package_TO_SOT_SMD:SOT-23, symbol Astra_Sequencing:BSS138LT1G
- added R311, R312, R313, R314, R315, R350, R351, R352, R353, R354, R355, R356, R357, R358, R359, R360, R361, R362, R363, R364, R365, R366, R367, R368, R369, R370, R391, R393, R395: 100k, Resistor_SMD:R_0603_1608Metric, symbol Astra_Sequencing:R
- added R340, R380, R381, R382, R390, R392, R394: 10.0k, Resistor_SMD:R_0603_1608Metric, symbol Astra_Sequencing:R
- added TP237: DOWNSTREAM_RUN_DELAYED, TestPoint:TestPoint_Pad_D1.0mm, symbol Astra_Sequencing:TestPoint
- added TP238: DOWNSTREAM_EN, TestPoint:TestPoint_Pad_D1.0mm, symbol Astra_Sequencing:TestPoint
- added TP239: SEQ_RUN_Q, TestPoint:TestPoint_Pad_D1.0mm, symbol Astra_Sequencing:TestPoint
- added TP240: SEQ_SHUT, TestPoint:TestPoint_Pad_D1.0mm, symbol Astra_Sequencing:TestPoint
- added TP241: SYS_HWRST, TestPoint:TestPoint_Pad_D1.0mm, symbol Astra_Sequencing:TestPoint
- added TP242: SYS_HWRST_CLEAN, TestPoint:TestPoint_Pad_D1.0mm, symbol Astra_Sequencing:TestPoint
- added TP243: AMP_FAULT_N, TestPoint:TestPoint_Pad_D1.0mm, symbol Astra_Sequencing:TestPoint
- added TP244: AMP_FAULT_CLEAN_N, TestPoint:TestPoint_Pad_D1.0mm, symbol Astra_Sequencing:TestPoint
- added TP245: SAFE_HW_CLEAR_N, TestPoint:TestPoint_Pad_D1.0mm, symbol Astra_Sequencing:TestPoint
- added TP246: SAFE_CLEAR_N, TestPoint:TestPoint_Pad_D1.0mm, symbol Astra_Sequencing:TestPoint
- added TP247: HW_RUN_LATCHED, TestPoint:TestPoint_Pad_D1.0mm, symbol Astra_Sequencing:TestPoint
- added TP248: ANALOG_PWR_EN, TestPoint:TestPoint_Pad_D1.0mm, symbol Astra_Sequencing:TestPoint
- added TP249: CLOCK_STARTUP_EN, TestPoint:TestPoint_Pad_D1.0mm, symbol Astra_Sequencing:TestPoint
- added TP250: AUDIO_DATA_OE_RELEASE, TestPoint:TestPoint_Pad_D1.0mm, symbol Astra_Sequencing:TestPoint
- added TP251: RUN_HEALTH_OK_3V8, TestPoint:TestPoint_Pad_D1.0mm, symbol Astra_Sequencing:TestPoint
- added TP252: ADC_PD_RST_N, TestPoint:TestPoint_Pad_D1.0mm, symbol Astra_Sequencing:TestPoint
- added TP253: SHUTDOWN_REQ_3V8, TestPoint:TestPoint_Pad_D1.0mm, symbol Astra_Sequencing:TestPoint
- added TP254: SAFE_ARM_3V8, TestPoint:TestPoint_Pad_D1.0mm, symbol Astra_Sequencing:TestPoint
- added TP255: 3V8_PRE, TestPoint:TestPoint_Pad_D1.0mm, symbol Astra_Sequencing:TestPoint
- added TP256: POWER_GND, TestPoint:TestPoint_Pad_D1.0mm, symbol Astra_Sequencing:TestPoint
- added U212, U213, U214, U215, U216, U217, U218, U219, U220: SN74LV1T08DBVR, Package_TO_SOT_SMD:SOT-23-5, symbol Astra_Sequencing:SN74LV1T08DBVR
- added U221, U222: SN74LVC1G74DCUR, Package_SO:VSSOP-8_2.3x2mm_P0.5mm, symbol Astra_Sequencing:SN74LVC1G74DCUR
- added U223: SN74LVC2G17DBVR, Package_TO_SOT_SMD:SOT-23-6, symbol Astra_Sequencing:SN74LVC2G17DBVR
- added U224, U229: SN74LVC2G07DBVR, Package_TO_SOT_SMD:SOT-23-6, symbol Astra_Sequencing:SN74LVC2G07DBVR
- added U225: TPS3760E012DYYR, Astra_Sequencing:Texas_DYY0014A, symbol Astra_Sequencing:TPS3760E012DYYR
- added U226: SN74LXC8T245PWR, Package_SO:TSSOP-24_4.4x7.8mm_P0.65mm, symbol Astra_Sequencing:SN74LXC8T245PWR
- added U227, U228: SN74LVC2G08DCUR, Package_SO:VSSOP-8_2.3x2mm_P0.5mm, symbol Astra_Sequencing:SN74LVC2G08DCUR
- added U230, U231, U232, U233, U234, U235, U236, U237, U238, U239, U240, U241, U242, U243: TMUX2821DSGR, Package_DFN_QFN:DFN-8-1EP_2x2mm_P0.5mm_EP0.9x1.6mm, symbol Astra_Sequencing:TMUX2821DSGR
- TP201, TP202, TP203, TP204, TP205, TP206, TP207, TP208, TP209, TP210, TP211, TP212, TP213, TP214, TP215, TP216, TP217, TP218, TP219, TP220, TP221, TP222, TP223, TP224, TP225, TP226, TP227, TP228: footprint (none) -> TestPoint:TestPoint_Pad_D1.0mm
- TP229: value EN_3V3_SYS -> MCLK_OE_N; footprint (none) -> TestPoint:TestPoint_Pad_D1.0mm
- TP230: value AFE_EN -> AUDIO_CLOCK_OE_N; footprint (none) -> TestPoint:TestPoint_Pad_D1.0mm
- TP231: value PGOOD_12V -> AUDIO_DATA_OE_N; footprint (none) -> TestPoint:TestPoint_Pad_D1.0mm
- TP232: value EFUSE_FLT_N -> PGOOD_12V; footprint (none) -> TestPoint:TestPoint_Pad_D1.0mm
- TP233: value 12V_PROTECTED -> PGOOD_CLEAN; footprint (none) -> TestPoint:TestPoint_Pad_D1.0mm
- TP234: value POWER_GND -> EFUSE_FLT_N; footprint (none) -> TestPoint:TestPoint_Pad_D1.0mm
- TP235: value SUP_REF -> EFUSE_FLT_CLEAN_N; footprint (none) -> TestPoint:TestPoint_Pad_D1.0mm
- TP236: value AFE_EN_CMD -> OUT1; footprint (none) -> TestPoint:TestPoint_Pad_D1.0mm
- U211: Authority (none) -> Phase 3E + Phase 3F; Function (none) -> Downstream qualification 1/2
Connections:
- net AFE_EN_CMD is gone; now on net OUT1: TP236.1
- net 12V_PROTECTED: no longer TP233.1
- net 1V8_DSP_REF_ANA: now also R390.1
- net 2V8_MIC: now also C360.1, C362.1, U240.8 (VDD), U242.8 (VDD)
- net 3V3_ADC_A: now also C351.1, C353.1, C355.1, C357.1, C358.1, U231.8 (VDD), U233.8 (VDD), U235.8 (VDD), U237.8 (VDD), U238.8 (VDD)
- net 3V3_SYS: now also C316.1, C318.1, C341.1, R380.1, R381.1, R392.1, R394.1, U226.1 (VCCA), U226.2 (DIR), U227.8 (VCC), U229.5 (VCC)
- net 3V8_PRE: now also C300.1, C301.1, C302.1, C303.1, C304.1, C305.1, C306.1, C307.1, C308.1, C309.1, C310.1, C311.1, C312.1, C313.1, C314.1, C315.1, C317.1, R340.1, R382.1, TP255.1, U212.5 (VCC), U213.5 (VCC), U214.5 (VCC), U215.5 (VCC), U216.5 (VCC), U217.5 (VCC), U218.5 (VCC), U219.5 (VCC), U220.5 (VCC), U221.6 (~{CLR}), U221.8 (VCC), U222.2 (D), U222.7 (~{PRE}), U222.8 (VCC), U223.5 (VCC), U224.5 (VCC), U225.1 (VDD), U226.23 (VCCB), U226.24 (VCCB), U228.8 (VCC)
- net 5V_AFE: now also C350.1, C352.1, C354.1, C356.1, C359.1, C361.1, C363.1, U230.8 (VDD), U232.8 (VDD), U234.8 (VDD), U236.8 (VDD), U239.8 (VDD), U241.8 (VDD), U243.8 (VDD)
- net EFUSE_FLT_N: now also TP234.1, R382.2, U223.3 (2A); no longer TP232.1
- net OUT1: no longer U202.8 (EN), U205.5 (EN), U207.3 (EN), U208.3 (EN)
- net PGOOD_12V: now also TP232.1, U223.1 (1A); no longer TP231.1, U211.2 (B)
- net POWER_GND: now also C300.2, C301.2, C302.2, C303.2, C304.2, C305.2, C306.2, C307.2, C308.2, C309.2, C310.2, C311.2, C312.2, C313.2, C314.2, C315.2, C316.2, C317.2, C318.2, C340.2, C341.2, C350.2, C351.2, C352.2, C353.2, C354.2, C355.2, C356.2, C357.2, C358.2, C359.2, C360.2, C361.2, C362.2, C363.2, Q201.2 (S), Q202.2 (S), Q203.2 (S), R311.2, R312.2, R313.2, R314.2, R315.2, R350.2, R351.2, R352.2, R353.2, R354.2, R355.2, R356.2, R357.2, R358.2, R359.2, R360.2, R361.2, R362.2, R363.2, R364.2, R365.2, R366.2, R367.2, R368.2, R369.2, R370.2, R391.2, R393.2, R395.2, TP256.1, U212.3 (GND), U213.3 (GND), U214.3 (GND), U215.3 (GND), U216.3 (GND), U217.3 (GND), U218.3 (GND), U219.3 (GND), U220.3 (GND), U221.2 (D), U221.4 (GND), U222.4 (GND), U223.2 (GND), U224.2 (GND), U225.13 (GND), U225.8 (GND), U226.11 (GND), U226.12 (GND), U226.13 (GND), U226.22 (~{OE}), U227.4 (GND), U228.4 (GND), U229.2 (GND), U230.4 (GND), U230.9 (EP), U231.4 (GND), U231.9 (EP), U232.4 (GND), U232.9 (EP), U233.4 (GND), U233.9 (EP), U234.4 (GND), U234.9 (EP), U235.4 (GND), U235.9 (EP), U236.4 (GND), U236.9 (EP), U237.4 (GND), U237.9 (EP), U238.3 (SEL2), U238.4 (GND), U238.9 (EP), U239.3 (SEL2), U239.4 (GND), U239.9 (EP), U240.4 (GND), U240.9 (EP), U241.4 (GND), U241.9 (EP), U242.4 (GND), U242.9 (EP), U243.4 (GND), U243.9 (EP); no longer TP234.1
- net RAILS_OK: now also Q201.1 (G), R391.1
- net SUP_REF: no longer TP235.1
- net SYS_HWRST: now also R356.1, TP241.1, U224.4 (2Y), U224.6 (1Y), U226.9 (A7), U229.1 (1A)
- net AFE_EN renamed ANALOG_PWR_EN
- net ANALOG_PWR_EN: now also U208.3 (EN), R311.1, TP248.1, U219.4 (Y), U230.3 (SEL2), U230.7 (SEL1), U231.3 (SEL2), U231.7 (SEL1), U232.3 (SEL2), U232.7 (SEL1), U233.3 (SEL2), U233.7 (SEL1), U234.3 (SEL2), U234.7 (SEL1), U235.3 (SEL2), U235.7 (SEL1), U236.3 (SEL2), U236.7 (SEL1), U237.3 (SEL2), U237.7 (SEL1), U238.7 (SEL1), U239.7 (SEL1), U240.3 (SEL2), U240.7 (SEL1), U241.3 (SEL2), U241.7 (SEL1), U242.3 (SEL2), U242.7 (SEL1), U243.3 (SEL2), U243.7 (SEL1); no longer TP230.1
- removed net EN_3V3_SYS: TP229.1, U203.8 (EN), U211.4 (Y)
- new net ADC_AIN1N: U231.6 (D2)
- new net ADC_AIN1P: U231.2 (D1)
- new net ADC_AIN2N: U233.6 (D2)
- new net ADC_AIN2P: U233.2 (D1)
- new net ADC_AIN3N: U235.6 (D2)
- new net ADC_AIN3P: U235.2 (D1)
- new net ADC_AIN4N: U237.6 (D2)
- new net ADC_AIN4P: U237.2 (D1)
- new net ADC_PD_RST_N: R381.2, TP252.1, U229.4 (2Y), U229.6 (1Y)
- new net ADC_RST_RELEASE_CMD: R368.1, U229.3 (2A)
- new net ADC_VREF: U238.1 (S1)
- new net AFE1N_AFTER_47R: U230.5 (S2)
- new net AFE1P_AFTER_47R: U230.1 (S1)
- new net AFE1_BEFORE_4u7: U241.2 (D1)
- new net AFE2N_AFTER_47R: U232.5 (S2)
- new net AFE2P_AFTER_47R: U232.1 (S1)
- new net AFE2_BEFORE_4u7: U241.6 (D2)
- new net AFE3N_AFTER_47R: U234.5 (S2)
- new net AFE3P_AFTER_47R: U234.1 (S1)
- new net AFE3_BEFORE_4u7: U243.2 (D1)
- new net AFE4N_AFTER_47R: U236.5 (S2)
- new net AFE4P_AFTER_47R: U236.1 (S1)
- new net AFE4_BEFORE_4u7: U243.6 (D2)
- new net AFE_VCM_INPUT: U239.2 (D1)
- new net AMP_FAULT_CLEAN_N: R365.1, TP244.1, U215.2 (B), U226.14 (B8)
- new net AMP_FAULT_N: R357.1, R380.2, TP243.1, U226.10 (A8)
- new net AMP_MUTE_CMD: R366.1, U227.2 (1B)
- new net AMP_MUTE_RELEASE: R369.1, U227.7 (1Y)
- new net AMP_STBY_CMD: R367.1, U227.6 (2B)
- new net AMP_STBY_RELEASE: R370.1, U227.3 (2Y)
- new net ANALOG_PERMIT: U218.4 (Y), U219.1 (A)
- new net ANALOG_PWR_CMD: R352.1, U226.5 (A3)
- new net ANALOG_PWR_CMD_3V8: R360.1, U219.2 (B), U226.19 (B3)
- new net AUDIO_CLOCK_OE_N: Q202.3 (D), R392.2, TP230.1
- new net AUDIO_DATA_OE_CMD: R354.1, U226.7 (A5)
- new net AUDIO_DATA_OE_CMD_3V8: R362.1, U220.2 (B), U226.17 (B5)
- new net AUDIO_DATA_OE_N: Q203.3 (D), R394.2, TP231.1
- new net AUDIO_DATA_OE_RELEASE: Q203.1 (G), R395.1, TP250.1, U220.4 (Y)
- new net CLOCK_STARTUP_CMD: R353.1, U226.6 (A4)
- new net CLOCK_STARTUP_CMD_3V8: R361.1, U226.18 (B4), U228.2 (1B)
- new net CLOCK_STARTUP_EN: Q202.1 (G), R393.1, TP249.1, U228.7 (1Y)
- new net DOWNSTREAM_EN: R312.1, R313.1, R314.1, R315.1, TP238.1, U202.8 (EN), U203.8 (EN), U205.5 (EN), U207.3 (EN), U212.4 (Y), U218.1 (A)
- new net DOWNSTREAM_RUN_DELAYED: R340.2, TP237.1, U212.2 (B), U225.6 (~{RESET})
- new net DOWNSTREAM_VALID: U211.4 (Y), U212.1 (A)
- new net DOWN_CTS: C340.1, U225.10 (CTS)
- new net EFUSE_FLT_CLEAN_N: TP235.1, U215.1 (A), U223.4 (2Y)
- new net HW_RUN_LATCHED: TP247.1, U218.2 (B), U220.1 (A), U222.5 (Q), U227.1 (1A), U227.5 (2A)
- new net ISO_0_0: U230.2 (D1), U231.1 (S1)
- new net ISO_0_1: U230.6 (D2), U231.5 (S2)
- new net ISO_1_0: U232.2 (D1), U233.1 (S1)
- new net ISO_1_1: U232.6 (D2), U233.5 (S2)
- new net ISO_2_0: U234.2 (D1), U235.1 (S1)
- new net ISO_2_1: U234.6 (D2), U235.5 (S2)
- new net ISO_3_0: U236.2 (D1), U237.1 (S1)
- new net ISO_3_1: U236.6 (D2), U237.5 (S2)
- new net ISO_4_0: U238.2 (D1), U239.1 (S1)
- new net ISO_5_0: U240.2 (D1), U241.1 (S1)
- new net ISO_5_1: U240.6 (D2), U241.5 (S2)
- new net ISO_6_0: U242.2 (D1), U243.1 (S1)
- new net ISO_6_1: U242.6 (D2), U243.5 (S2)
- new net MCLK_OE_N: Q201.3 (D), R390.2, TP229.1
- new net MIC1_AFTER_100R: U240.1 (S1)
- new net MIC2_AFTER_100R: U240.5 (S2)
- new net MIC3_AFTER_100R: U242.1 (S1)
- new net MIC4_AFTER_100R: U242.5 (S2)
- new net PGOOD_CLEAN: TP233.1, U211.2 (B), U213.2 (B), U214.1 (A), U221.7 (~{PRE}), U223.6 (1Y), U224.3 (2A)
- new net RUN_HEALTH_OK_3V8: R363.1, TP251.1, U226.16 (B6), U228.6 (2B)
- new net RUN_HEALTH_OK_CMD: R355.1, U226.8 (A6)
- new net SAFE_ARM_3V8: TP254.1, U217.4 (Y), U222.1 (CLK)
- new net SAFE_ARM_CMD: R351.1, U226.4 (A2)
- new net SAFE_ARM_CMD_3V8: R359.1, U217.1 (A), U226.20 (B2)
- new net SAFE_CLEAR_N: TP246.1, U222.6 (~{CLR}), U228.3 (2Y)
- new net SAFE_FAULTS: U215.4 (Y), U216.2 (B)
- new net SAFE_HW_CLEAR_N: TP245.1, U216.4 (Y), U228.5 (2A)
- new net SAFE_PWR_RESET: U214.4 (Y), U216.1 (A)
- new net SEQ_RUN_Q: TP239.1, U221.5 (Q), U224.1 (1A)
- new net SEQ_SHUT: TP240.1, U221.3 (~{Q}), U225.3 (SENSE)
- new net SHUTDOWN_CLK_3V8: U213.4 (Y), U221.1 (CLK)
- new net SHUTDOWN_REQ: R350.1, U226.3 (A1)
- new net SHUTDOWN_REQ_3V8: R358.1, TP253.1, U213.1 (A), U226.21 (B1)
- new net SYS_HWRST_CLEAN: R364.1, TP242.1, U214.2 (B), U217.2 (B), U226.15 (B7), U228.1 (1A)
- no-connect marks 15 -> 28
Other:
- note added: "ADC VREF -> AFE VCM buffer; spare channels OFF"
- note added: "ADC reset: system reset AND deliberate release"
- note added: "AFE channel 1 -> ADC, two differential legs"
- note added: "AFE channel 2 -> ADC, two differential legs"
- note added: "AFE channel 3 -> ADC, two differential legs"
- note added: "AFE channel 4 -> ADC, two differential legs"
- note added: "Amplifier MUTE / STANDBY authorization"
- note added: "Analog qualification 1/2"
- note added: "Analog qualification 2/2"
- note added: "CTS 198..242nF acceptance: hold 20.415..40.946ms. CTR/MR open. Cold-start reset may add <=2ms."
- note added: "Commanded shutdown clock"
- note added: "Data authorization; no bootstrap gating"
- note added: "Downstream qualification 1/2"
- note added: "Downstream qualification 2/2"
- note added: "Explicit post-check arm edge"
- note added: "Hardware safe clear 1/3"
- note added: "Hardware safe clear 2/3"
- note added: "Hardware safe clear 3/3"
- note added: "MCLK /OE from RAILS_OK only. Clock bank /1OE from CLOCK_STARTUP_EN. Data bank /2OE from AUDIO_DATA_OE_RELEASE only. SN74AXC2T245, LVC244A, ASDLJ/LMK and endpoints: later-sheet contracts. ADC sheet: DVDD CEXT=10uF X7R, Ceff<=12uF, REXT=3.00k 1%; PD/RST LOW >=50ms for in-place reset; PWUP only after DVDD+clock >=10ms."
- note added: "Microphone pair 1 -> AFE coupling capacitors"
- note added: "Microphone pair 2 -> AFE coupling capacitors"
- note added: "P variant: active output discharge. Qualified branch EN. No startup-time guarantee extrapolated to this capacitor bank. Consumer-side filtering/decoupling belongs to the later load sheets."
- note added: "Raw PGOOD / eFuse Schmitt conditioning"
- note added: "Retained shutdown / immediate brownout reset"
- note added: "START: RAILS_OK -> MCLK -> DSP boot -> CLOCK_STARTUP_CMD -> ADC reset/config/PLL -> RUN_HEALTH_OK + arm edge. Only after arm: data, amplifier Hi-Z clock check, analog settling, then MUTE/PLAY. ADC-only PLL loss: hardware automute + firmware health withdrawal. STOP: MUTE/Hi-Z/STANDBY >=15ms -> analog OFF, >=1ms -> data OFF + ADC reset -> health LOW -> clock command LOW -> SHUTDOWN_REQ. Retained re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"
- note added: "U_BOOT_GATES: clock bootstrap / health clear"
- note added: "U_CMD_XLAT: eight isolated A-to-B controls"
- note added: "U_DOWN_DELAY: OV / active-low / open drain"
- note added: "U_SAFE_LATCH: functional authorization"
- note added: "U_SEQ_RUN: retained service-off state"
- note added: "Used SEL = ANALOG_PWR_EN; either adjacent rail absent isolates path. No endpoint load circuitry. Keep differential switch paths symmetrical."
- note removed: "3V3_SYS EN = OUT1 AND PGOOD_12V 1.0M EN pulldown; inputs remain separate status nets."
- note removed: "AFE EN held off by R310. Command and fault override NOT connected. No power-up / reset / safe-state implementation approval is implied. Hardware-safe latch, dominance, commanded shutdown, and AFE override are incomplete."
- note removed: "P variant: active output discharge. EN=OUT1. No startup-time guarantee extrapolated to this capacitor bank. Consumer-side filtering/decoupling belongs to the later load sheets."
- note removed: "PHASE 4B BLOCKED: common OUT1 cannot turn microphones off while retaining core/DMC power. Phase 3D section 9.1(5), 11(6) versus section 9.2 commanded-shutdown order. No enable relation changed."
- moved on the sheet: R310, TP229, TP230, TP231, TP232, TP233, TP234, TP235, TP236, U211

Commit message: before-rebuilding
Last changes before rebuilding PCB design
Parts:
- removed U240, U241, U242, U243: TMUX2821DSGR, Package_DFN_QFN:DFN-8-1EP_2x2mm_P0.5mm_EP0.9x1.6mm, symbol Astra_Sequencing:TMUX2821DSGR
- added U240, U241, U242, U243: TMUX1574PWR, Package_SO:TSSOP-16_4.4x5mm_P0.65mm, symbol Astra_Sequencing:TMUX1574PWR
Connections:
- net 2V8_MIC: now also U240.16 (VDD), U242.16 (VDD)
- net 5V_AFE: now also U241.16 (VDD), U243.16 (VDD)
- net POWER_GND: now also U240.1 (SEL), U240.10 (S3B), U240.13 (S4B), U240.15 (EN), U240.3 (S1B), U240.6 (S2B), U240.8 (GND), U241.1 (SEL), U241.10 (S3B), U241.13 (S4B), U241.15 (EN), U241.3 (S1B), U241.6 (S2B), U241.8 (GND), U242.1 (SEL), U242.10 (S3B), U242.13 (S4B), U242.15 (EN), U242.3 (S1B), U242.6 (S2B), U242.8 (GND), U243.1 (SEL), U243.10 (S3B), U243.13 (S4B), U243.15 (EN), U243.3 (S1B), U243.6 (S2B), U243.8 (GND)
- net ADC_AIN1N renamed ADC1_N_ISO
- net ADC_AIN1P renamed ADC1_P_ISO
- net ADC_AIN2N renamed ADC2_N_ISO
- net ADC_AIN2P renamed ADC2_P_ISO
- net ADC_AIN3N renamed ADC3_N_ISO
- net ADC_AIN3P renamed ADC3_P_ISO
- net ADC_AIN4N renamed ADC4_N_ISO
- net ADC_AIN4P renamed ADC4_P_ISO
- net ADC_VREF renamed ADC_VREF_RAW
- net AFE1N_AFTER_47R renamed AFE1_N_RAW
- net AFE1P_AFTER_47R renamed AFE1_P_RAW
- net AFE2N_AFTER_47R renamed AFE2_N_RAW
- net AFE2P_AFTER_47R renamed AFE2_P_RAW
- net AFE3N_AFTER_47R renamed AFE3_N_RAW
- net AFE3P_AFTER_47R renamed AFE3_P_RAW
- net AFE4N_AFTER_47R renamed AFE4_N_RAW
- net AFE4P_AFTER_47R renamed AFE4_P_RAW
- net AFE_VCM_INPUT renamed AFE_VCM_ISO
- new net MIC1_N_ISO: U241.7 (D2)
- new net MIC1_N_MID: U240.7 (D2), U241.5 (S2A)
- new net MIC1_N_RAW: U240.5 (S2A)
- new net MIC1_P_ISO: U241.4 (D1)
- new net MIC1_P_MID: U240.4 (D1), U241.2 (S1A)
- new net MIC1_P_RAW: U240.2 (S1A)
- new net MIC2_N_ISO: U241.12 (D4)
- new net MIC2_N_MID: U240.12 (D4), U241.14 (S4A)
- new net MIC2_N_RAW: U240.14 (S4A)
- new net MIC2_P_ISO: U241.9 (D3)
- new net MIC2_P_MID: U240.9 (D3), U241.11 (S3A)
- new net MIC2_P_RAW: U240.11 (S3A)
- new net MIC3_N_ISO: U243.7 (D2)
- new net MIC3_N_MID: U242.7 (D2), U243.5 (S2A)
- new net MIC3_N_RAW: U242.5 (S2A)
- new net MIC3_P_ISO: U243.4 (D1)
- new net MIC3_P_MID: U242.4 (D1), U243.2 (S1A)
- new net MIC3_P_RAW: U242.2 (S1A)
- new net MIC4_N_ISO: U243.12 (D4)
- new net MIC4_N_MID: U242.12 (D4), U243.14 (S4A)
- new net MIC4_N_RAW: U242.14 (S4A)
- new net MIC4_P_ISO: U243.9 (D3)
- new net MIC4_P_MID: U242.9 (D3), U243.11 (S3A)
- new net MIC4_P_RAW: U242.11 (S3A)
Other:
- note added: "Phase 3G: MIC1/2 P,N; EN=SEL=0; spare SxB grounded; rail-off isolation."
- note added: "Phase 3G: MIC3/4 P,N; EN=SEL=0; spare SxB grounded; rail-off isolation."
- note removed: "Microphone pair 1 -> AFE coupling capacitors"
- note removed: "Microphone pair 2 -> AFE coupling capacitors"
